Commit message: Imported upstream version '0.6.8' of 'upstream'

File: cob_gazebo_worlds/urdf/ipa-apartment/ipa-apartment.urdf.xacro (robot description, xacro)
@@ -19,17 +19,17 @@
   <xacro:include filename="$(find cob_gazebo_worlds)/urdf/ipa-apartment/wall_ipa.urdf.xacro" />
   <!--Parameters-->
-  <property name="dist_axis_x" value="1.969" />
-  <property name="dist_axis_y" value="4.070" />
-  <property name="size_total_x" value="8.0" />
-  <property name="size_total_y" value="11.2" />
-  <property name="size_a" value="4.7" />
-  <property name="size_b" value="8.2" />
-  <property name="size_c" value="1.8" />
-  <property name="size_d" value="4.16" />
-  <property name="wall_depth" value="0.1" />
-  <property name="window_depth" value="0.15" />
-  <property name="size_z_wall1" value="2.7" />
-  <property name="size_z_wall2" value="2.7" />
-  <property name="size_z_wall3" value="2.7" />
+  <xacro:property name="dist_axis_x" value="1.969" />
+  <xacro:property name="dist_axis_y" value="4.070" />
+  <xacro:property name="size_total_x" value="8.0" />
+  <xacro:property name="size_total_y" value="11.2" />
+  <xacro:property name="size_a" value="4.7" />
+  <xacro:property name="size_b" value="8.2" />
+  <xacro:property name="size_c" value="1.8" />
+  <xacro:property name="size_d" value="4.16" />
+  <xacro:property name="wall_depth" value="0.1" />
+  <xacro:property name="window_depth" value="0.15" />
+  <xacro:property name="size_z_wall1" value="2.7" />
+  <xacro:property name="size_z_wall2" value="2.7" />
+  <xacro:property name="size_z_wall3" value="2.7" />
   <xacro:macro name="ipa-apartment" params="name">
     <gazebo>
@@ -51,6 +51,6 @@
     <xacro:cabinets name="cabinets">
     </xacro:cabinets>
-    <xacro:kitchen name="kitchen">
-    </xacro:kitchen>
+    <!--xacro:kitchen name="kitchen">
+    </xacro:kitchen-->
     <xacro:wall_ipa name="wall_ipa">
     </xacro:wall_ipa>
